File: Testproject/testboard1.brd (EAGLE design)
At the start: 101.3 x 81.3 mm, 18 parts, among them U1 AD8232

Commit message: updated board design
updated board design
Parts:
- removed JP2: (no value), SparkFun-Connectors:AUDIO-JACK-3.5MM-SMD
- moved R1 6.48 mm to (45.7, 26.7), turned to 180 degrees
- moved D1 4.58 mm to (55.9, 36.8)
- moved JP1 4.02 mm to (39.4, 35.6), turned to 270 degrees
- moved R10 2.84 mm to (50.8, 35.6), turned to 270 degrees
- moved SJ4 2.84 mm to (55.9, 34.3), turned to 0 degrees
- moved R4 2.84 mm to (45.7, 31.8), turned to 180 degrees
- moved R11 2.54 mm to (48.3, 35.6), turned to 90 degrees
- moved R16 2.54 mm to (49.5, 38.1)
- moved R3 2.54 mm to (43.2, 35.6), turned to 90 degrees
- moved R14 1.80 mm to (55.9, 29.2), turned to 270 degrees
- moved C2 1.80 mm to (45.7, 29.2), turned to 0 degrees
- moved C7 1.80 mm to (53.3, 29.2), turned to 90 degrees
- moved R5 1.27 mm to (41.9, 26.7), turned to 180 degrees
- moved C5 1.27 mm to (53.3, 35.6)
- turned C4 to 90 degrees
Connections:
- net LA: no longer JP2.RING
- net RA: no longer JP2.SLEEVE
- net RL: no longer JP2.TIP
Routing:
- net N$1: track 4.54 -> 33.8 mm
- net RL: track 12.5 -> 0.00 mm
- net N$5: track 21.6 -> 12.8 mm, vias 0 -> 2
- net RA: track 24.9 -> 18.1 mm, vias 0 -> 1
- net SIGNAL_OUT: track 35.2 -> 29.3 mm, vias 0 -> 2
- net N$10: track 6.30 -> 2.56 mm
- net GND: track 19.6 -> 16.5 mm
- net N$6: track 2.27 -> 5.32 mm
- net N$2: track 3.65 -> 5.72 mm, vias 0 -> 2
- net N$18: track 9.34 -> 7.77 mm
- net 3.3V: track 11.2 -> 9.79 mm
- net N$13: track 5.33 -> 4.02 mm
- net N$4: track 6.88 -> 5.75 mm
- net LA: vias 0 -> 1
