File: Testproject/testboard1.sch (EAGLE design)
At the start: 18 parts, among them U1 AD8232

Commit message: updated board design
updated board design
Parts:
- removed JP2: (no value), SparkFun-Connectors:AUDIO-JACKSMD2
Connections:
- net LA: no longer JP2.RIGHT
- net RA: no longer JP2.SLEEVE
- net RL: no longer JP2.LEFT
Changed lines of the file:
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@@
 <part name="GND2" library="SparkFun-Aesthetics" deviceset="GND" device=""/>
 <part name="SUPPLY3" library="SparkFun-Aesthetics" deviceset="3.3V" device=""/>
-<part name="JP2" library="SparkFun-Connectors" deviceset="AUDIO-JACK" device="SMD2"/>
 <part name="JP1" library="SparkFun-Connectors" deviceset="M03" device="PTH"/>
 <part name="R16" library="SparkFun-Resistors" deviceset="1K-1%" device="" value="1k"/>
@@
 <attribute name="VALUE" x="167.894" y="92.456" size="1.778" layer="96"/>
 </instance>
-<instance part="JP2" gate="G$1" x="205.74" y="172.72" smashed="yes" rot="R270">
-<attribute name="NAME" x="208.788" y="177.8" size="1.778" layer="95" rot="R270"/>
-<attribute name="VALUE" x="200.66" y="177.8" size="1.778" layer="96" rot="R270"/>
-</instance>
 <instance part="JP1" gate="G$1" x="205.74" y="144.78" smashed="yes" rot="R270">
 <attribute name="VALUE" x="198.12" y="147.32" size="1.778" layer="96" rot="R270"/>
@@
 </segment>
 <segment>
-<pinref part="JP2" gate="G$1" pin="RIGHT"/>
-<wire x1="205.74" y1="167.64" x2="205.74" y2="162.56" width="0.1524" layer="91"/>
-<label x="205.74" y="162.56" size="1.27" layer="95" rot="R270" xref="yes"/>
-</segment>
-<segment>
 <wire x1="205.74" y1="137.16" x2="205.74" y2="134.62" width="0.1524" layer="91"/>
 <label x="205.74" y="134.62" size="1.27" layer="95" rot="R270" xref="yes"/>
@@
 <wire x1="93.98" y1="119.38" x2="93.98" y2="124.46" width="0.1524" layer="91"/>
 <junction x="93.98" y="124.46"/>
-</segment>
-<segment>
-<pinref part="JP2" gate="G$1" pin="SLEEVE"/>
-<wire x1="208.28" y1="167.64" x2="208.28" y2="162.56" width="0.1524" layer="91"/>
-<label x="208.28" y="162.56" size="1.27" layer="95" rot="R270" xref="yes"/>
 </segment>
 <segment>
@@
 <net name="RL" class="0">
 <segment>
-<pinref part="JP2" gate="G$1" pin="LEFT"/>
-<wire x1="203.2" y1="167.64" x2="203.2" y2="162.56" width="0.1524" layer="91"/>
-<label x="203.2" y="162.56" size="1.27" layer="95" rot="R270" xref="yes"/>
-</segment>
-<segment>
 <wire x1="203.2" y1="137.16" x2="203.2" y2="134.62" width="0.1524" layer="91"/>
